Commit message: 텐던 장착 실측 기반 재캘리브레이션: 중립 1900 / flex 전채널 -1 / yaw 차동 / fspan 950
실물(텐던 연결 4손가락) 진단 결과 pitch 가 거의 안 나오던 원인 두 가지를 고친다.
- 텐던 슬랙: 중립 1500±480 설계에서는 굽힘이 ~1500us 아래에서야 시작, 최대 ~900us.
  중립을 1900(손가락 폄·텐던 막 팽팽)으로 올리고 flex 는 0..+ 한 방향이므로
  아래로 950us 를 전부 굽힘 행정으로 쓴다 (ES3352 스펙 800~2200us, 750 이하 끝단 고정).
- 부호: 두 서보 모두 낮은 us = 당김. flexSign 전채널 -1, yawSign Out +1 / In -1.

펌웨어(rev.4): 기본 캘리브 표·flexSpan 950·SPAN_MAX 1000, room() 을 단방향 flex 기준으로.
  EEPROM 8채널 저장 완료 (neutral 1900, fspan 950, yspan 150).
ROS: servo_map 미러·flex_span_us 950·pitch_max_rad 1.10(MCP 기준),
  URDF --pitch-limit 1.10, 충돌행렬/SRDF 재생성, 프리셋 pitch 상한 검지/중지/약지 1.05 ·
  소지 0.95 (모델 너클<->base_link 자기충돌 한계). verify_offline room 검사 단방향화.
검증: check_presets 12/12, verify_offline 0 실패, pytest 7, MoveIt 프리셋 실물 구동 확인.

Co-Authored-By: Claude Fable 5 <noreply@anthropic.com>

File: src/dexhand_moveit_config/config/dexhandv2_right_8servo.urdf (robot description, URDF)
Before this commit: robot dexhandv2_right_8servo, 26 links, 25 joints
Joints:
- joint R_Index_Pitch: limit lower=0.0 upper=0.950000 effort=1.5 velocity=3.0 -> lower=0.0 upper=1.100000 effort=1.5 velocity=3.0
- joint R_Middle_Pitch: limit lower=0.0 upper=0.950000 effort=1.5 velocity=3.0 -> lower=0.0 upper=1.100000 effort=1.5 velocity=3.0
- joint R_Pinky_Pitch: limit lower=0.0 upper=0.950000 effort=1.5 velocity=3.0 -> lower=0.0 upper=1.100000 effort=1.5 velocity=3.0
- joint R_Ring_Pitch: limit lower=0.0 upper=0.950000 effort=1.5 velocity=3.0 -> lower=0.0 upper=1.100000 effort=1.5 velocity=3.0
